File: KiCad/Esquemático Aviônica/_autosave-Esquemático inical aviônica Anhangá.sch (KiCad schematic (older format))
At the start: 20 parts, among them J1 Conn_01x06_Female, J2 Conn_01x06_Female, J3 Conn_01x12_Female, J4 Conn_01x12_Female, J5 Screw_Terminal_01x02, J6 Conn_01x06_Male, J7 Screw_Terminal_01x02, J8 Conn_01x07_Female, Q1 IRF7403, U1 ME620933

Commit message: Esquemático e Layout reformulados
Changed lines of the file:
@@
 Text GLabel 2300 4350 0    50   Input ~ 0
 D_OUTPUT_NÍQUEL
-Text GLabel 2300 4350 2    50   Input ~ 0
+Text GLabel 2550 4350 2    50   Input ~ 0
 D2
 Text GLabel 3350 3950 1    50   Input ~ 0
@@
 Text GLabel 4700 3350 0    50   Input ~ 0
 D8
+Wire Wire Line
+	2300 4350 2550 4350
 $EndSCHEMATC
