File: KiCad/Esquemático Aviônica/Esquemático inical aviônica Anhangá.kicad_pcb (KiCad board)
At the start: 2 copper layers, 65 x 90 mm, 21 parts, among them J1 Conn_01x06_Female, J2 Conn_01x06_Female, J3 Conn_01x12_Female, J4 Conn_01x12_Female, J5 Screw_Terminal_01x02, J6 Conn_01x06_Male, J7 Screw_Terminal_01x02, J8 Conn_01x02_Female, J9 Conn_01x06_Male, Q1 IRF7403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

Commit message: PCB Anhangá
Parts:
- moved J3 51.7 mm to (133.5, 69.0), turned to 0 degrees
- moved J2 50.3 mm to (119.2, 66.5), turned to 90 degrees
- moved BZ1 49.0 mm to (135.2, 113.2), turned to 270 degrees
- moved U1 45.9 mm to (108.0, 65.8), turned to 180 degrees
- moved C2 45.0 mm to (106.4, 75.9)
- moved C1 41.5 mm to (109.5, 70.4), turned to 0 degrees
- moved J7 38.2 mm to (97.8, 71.9)
- moved J5 37.1 mm to (97.8, 79.5)
- moved R2 36.6 mm to (97.4, 100.5), turned to 270 degrees
- moved R1 34.1 mm to (103.4, 105.2), turned to 90 degrees
- moved D1 31.3 mm to (104.4, 80.5), turned to 270 degrees
- moved R4 30.9 mm to (107.2, 101.4), turned to 0 degrees
- moved J8 28.6 mm to (129.9, 80.4), turned to 180 degrees
- moved R3 28.4 mm to (108.0, 79.5), turned to 270 degrees
- moved R5 24.0 mm to (97.5, 92.4)
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Connections:
- BZ1 pad 1: D8 -> 10
- J1 pad 2: VBAT -> 5V
- J3 pad 12: (no net) -> 10
- J3 pad 7: (no net) -> ANAL_INPUT_V_NÍQUEL
- J3 pad 8: (no net) -> CS
- J4 pad 1: CS -> (no net)
- J4 pad 6: ANAL_INPUT_V_NÍQUEL -> (no net)
- J4 pad 8: D2 -> (no net)
- J8 pad 1: SCL -> SDA
- J8 pad 2: SDA -> SCL
- R4 pad 2: D2 -> D8
Routing:
- net SDA: track 149.9 -> 60.8 mm, vias 2 -> 0
- net VBAT: track 154.4 -> 73.4 mm, vias 2 -> 0
- net CS: track 152.7 -> 77.1 mm
- net 5V: track 0.00 -> 73.0 mm
- net ANAL_INPUT_V_NÍQUEL: track 50.3 -> 100.4 mm
- net D2: track 42.7 -> 0.00 mm
- net SCL: track 102.1 -> 60.9 mm, vias 2 -> 0
- net VCC: track 110.8 -> 83.6 mm, vias 2 -> 0
- net D8: track 34.5 -> 10.9 mm
- net Net-(D1-Pad2): track 71.3 -> 52.8 mm
- net 10: track 0.00 -> 17.0 mm
- net MOSI: track 72.5 -> 56.7 mm, vias 2 -> 0
- net RST: track 15.2 -> 0.00 mm
- net SCK: track 57.8 -> 67.1 mm
- net MISO: track 66.5 -> 62.0 mm
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Other:
- board size 65 x 90 mm -> 65 x 90.2 mm

Commit message: Esquemático Novo
Parts:
- R1, R2, R3, R4, R5: footprint Resistor_THT:R_Axial_DIN0207_L6.3mm_D2.5mm_P5.08mm_Vertical -> Resistor_THT:R_Axial_DIN0207_L6.3mm_D2.5mm_P7.62mm_Horizontal
- moved R3 4.64 mm to (111.0, 76.0)
- moved R2 4.10 mm to (97.4, 104.7)
- moved R5 2.45 mm to (100.0, 92.5)
- moved R4 2.40 mm to (107.0, 99.0)
- moved R1 1.66 mm to (102.8, 106.7), turned to 0 degrees
- moved C3 1.64 mm to (104.0, 93.0)
- moved Q1 1.54 mm to (109.0, 90.0)
Routing:
- net Net-(D1-Pad2): track 52.8 -> 47.9 mm
- net Net-(C3-Pad1): track 17.7 -> 14.1 mm
- net D8: track 10.9 -> 7.61 mm
- net ANAL_INPUT_V_NÍQUEL: track 100.4 -> 97.7 mm
- net SDA: track 60.8 -> 58.2 mm
- net SCL: track 60.9 -> 59.0 mm
- net VBAT: track 73.4 -> 75.2 mm
- net 5V: track 73.0 -> 71.6 mm
- net VCC: track 83.6 -> 84.6 mm
- net MISO: track 62.0 -> 61.2 mm
- net 10: track 17.0 -> 17.8 mm
